File: Z180Mboard-v3.kicad_pcb (KiCad board)
At the start: 2 copper layers, 170.2 x 170.2 mm, 88 parts, among them J1 Conn_02x05_Odd_Even, J10 PS2-MINIDIN6-FEMALE-SINGLE, J11 Conn_02x04_Odd_Even, J12 Conn_01x06, J13 Conn_01x06, J14 Conn_02x10_Top_Bottom, J15 Conn_02x05_Odd_Even, J16 DB9_Female, J17 Conn_01x40, J18 Conn_02x17_Odd_Even, J19 Conn_01x03, J2 Conn_02x05_Odd_Even, J20 Conn_02x09_Odd_Even, J21 Conn_02x09_Odd_Even, J22 Conn_02x09_Odd_Even, J3 Conn_02x05_Odd_Even, J4 Conn_02x05_Odd_Even, J5 Conn_02x05_Odd_Even, J6 Conn_02x05_Odd_Even, J7 Conn_02x05_Odd_Even, J8 Conn_01x08, J9 PS2-MINIDIN6-FEMALE-SINGLE, SW1 SW_SPST, SW2 SW_Push, U1 Z8-L180-S180-180-PLCC-68, U10 74LVC245, U11 DS1307+, U12 WD37C65C-DIP44, U13 74HCT138, U14 74HCT00, U15 74HCT32, U16 74HCT32, U2 SST39SF040, U3 74AHCT138, U4 74AHCT139, U5 AS6C4008-55PCN, U6 AS6C4008-55PCN, U7 82C55A_PLCC, U8 74HCT138, U9 74AHCT151, X1 CXO_DIP8, X2 CXO_DIP8, Y1 Crystal

Commit message: v3: Hopefully the final revision for this attempt
Parts:
- added J23: Conn_02x13_Odd_Even, Connector_IDC:IDC-Header_2x13_P2.54mm_Vertical, F.Cu at (180.6, 176.3)
- added J25: Conn_01x16, Connector_PinHeader_2.54mm:PinHeader_1x16_P2.54mm_Horizontal, F.Cu at (201.7, 187.2)
- added J26: Conn_01x16, Connector_PinHeader_2.54mm:PinHeader_1x16_P2.54mm_Vertical, F.Cu at (201.7, 183.4)
- added J27: Conn_01x03_Male, Connector_PinHeader_2.54mm:PinHeader_1x03_P2.54mm_Vertical, F.Cu at (205.7, 183.4)
- J20, J21, J22: value Conn_02x09_Odd_Even -> Conn_02x10_Odd_Even; footprint Connector_PinSocket_2.54mm:PinSocket_2x09_P2.54mm_Vertical -> Connector_PinSocket_2.54mm:PinSocket_2x10_P2.54mm_Vertical
- moved J20 2.54 mm to (142.2, 128.8)
- moved J21 2.54 mm to (124.0, 128.8)
- moved J22 2.54 mm to (105.7, 128.8)
Connections:
- J1 pad 3: (no net) -> DC3
- J12 pad 5: (no net) -> DC3
- J13 pad 5: (no net) -> DC
- J2 pad 3: (no net) -> DC3
- J20 pad 1: D7 -> CLK
- J20 pad 10: SLOTCS2 -> A2
- J20 pad 11: D2 -> D3
- J20 pad 12: INT -> SLOTCS2
- J20 pad 13: D1 -> D2
- J20 pad 14: RD2 -> INT
- J20 pad 15: D0 -> D1
- J20 pad 16: RESET -> RD2
- J20 pad 17: WR2 -> D0
- J20 pad 18: GND -> RESET
- J20 pad 3: D6 -> D7
- J20 pad 4: A0 -> M1
- J20 pad 5: D5 -> D6
- J20 pad 6: A1 -> A0
- J20 pad 7: D4 -> D5
- J20 pad 8: A2 -> A1
- J20 pad 9: D3 -> D4
- J21 pad 1: D7 -> CLK
- J21 pad 10: SLOTCS0 -> A2
- J21 pad 11: D2 -> D3
- J21 pad 12: INT -> SLOTCS0
- J21 pad 13: D1 -> D2
- J21 pad 14: RD0 -> INT
- J21 pad 15: D0 -> D1
- J21 pad 16: RESET -> RD0
- J21 pad 17: WR0 -> D0
- J21 pad 18: GND -> RESET
- J21 pad 3: D6 -> D7
- J21 pad 4: A0 -> M1
- J21 pad 5: D5 -> D6
- J21 pad 6: A1 -> A0
- J21 pad 7: D4 -> D5
- J21 pad 8: A2 -> A1
- J21 pad 9: D3 -> D4
- J22 pad 1: D7 -> CLK
- J22 pad 10: SLOTCS1 -> A2
- J22 pad 11: D2 -> D3
- J22 pad 12: INT -> SLOTCS1
- J22 pad 13: D1 -> D2
- J22 pad 14: RD1 -> INT
- J22 pad 15: D0 -> D1
- J22 pad 16: RESET -> RD1
- J22 pad 17: WR1 -> D0
- J22 pad 18: GND -> RESET
- J22 pad 3: D6 -> D7
- J22 pad 4: A0 -> M1
- J22 pad 5: D5 -> D6
- J22 pad 6: A1 -> A0
- J22 pad 7: D4 -> D5
- J22 pad 8: A2 -> A1
- J22 pad 9: D3 -> D4
- J3 pad 3: (no net) -> DC3
- J4 pad 3: (no net) -> DC3
- J5 pad 3: (no net) -> DC3
Routing:
- net DC3: track 0.00 -> 95.1 mm, vias 0 -> 1
- net M1: track 123.6 -> 190.7 mm, vias 0 -> 2
- net CLK: track 120.3 -> 179.8 mm, vias 1 -> 2
- net GND: track 1344.3 -> 1396.2 mm, vias 36 -> 51
- net TRK00: track 55.0 -> 98.9 mm, vias 0 -> 1
- net VCC: track 1199.1 -> 1240.3 mm
- net MOTEA: track 44.5 -> 81.2 mm, vias 2 -> 4
- net WPT: track 62.2 -> 97.2 mm
- net SIDE1: track 12.6 -> 44.9 mm, vias 0 -> 1
- net DRVSA: track 45.1 -> 77.3 mm, vias 1 -> 2
- net DC: track 144.1 -> 172.8 mm
- net RDATA: track 36.9 -> 64.6 mm, vias 0 -> 2
- net WGATE: track 27.4 -> 55.0 mm, vias 1 -> 2
- net STEP: track 30.6 -> 56.9 mm, vias 1 -> 2
- net INDEX: track 79.9 -> 99.8 mm
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Other:
- board text added: "Z180 MiniITX v3 (C) 2022 Alan Cox"
- board text removed: "PUT BACK THE MOUNTING HOLES"
- board text removed: "Z180 MiniITX v3 (C) 2020 Alan Cox"
