File: Z180Mboard-v3.sch (KiCad schematic (older format))
At the start: 88 parts, among them J1 Conn_02x05_Odd_Even, J10 PS2-MINIDIN6-FEMALE-SINGLE, J11 Conn_02x04_Odd_Even, J12 Conn_01x06, J13 Conn_01x06, J14 Conn_02x10_Top_Bottom, J15 Conn_02x05_Odd_Even, J16 DB9_Female, J17 Conn_01x40, J18 Conn_02x17_Odd_Even, J19 Conn_01x03, J2 Conn_02x05_Odd_Even, J20 Conn_02x09_Odd_Even, J21 Conn_02x09_Odd_Even, J22 Conn_02x09_Odd_Even, J3 Conn_02x05_Odd_Even, J4 Conn_02x05_Odd_Even, J5 Conn_02x05_Odd_Even, J6 Conn_02x05_Odd_Even, J7 Conn_02x05_Odd_Even, J8 Conn_01x08, J9 PS2-MINIDIN6-FEMALE-SINGLE, SW1 SW_SPST, SW2 SW_Push, U1 Z8-L180-S180-180-PLCC-68, U10 74LVC245, U11 DS1307+, U12 WD37C65C-DIP44, U13 74HCT138, U14 74HCT00, U15 74HCT32, U16 74HCT32, U2 SST39SF040, U3 74AHCT138, U4 74AHCT139, U5 AS6C4008-55PCN, U6 AS6C4008-55PCN, U7 82C55A_PLCC, U8 74HCT138, U9 74AHCT151, X1 CXO_DIP8, X2 CXO_DIP8, Y1 Crystal

Commit message: v3: Hopefully the final revision for this attempt
Parts:
- added J23: Conn_02x13_Odd_Even, Connector_IDC:IDC-Header_2x13_P2.54mm_Vertical, symbol Connector_Generic:Conn_02x13_Odd_Even
- added J25: Conn_01x16, Connector_PinHeader_2.54mm:PinHeader_1x16_P2.54mm_Horizontal, symbol Connector_Generic:Conn_01x16
- added J26: Conn_01x16, Connector_PinHeader_2.54mm:PinHeader_1x16_P2.54mm_Vertical, symbol Connector_Generic:Conn_01x16
- added J27: Conn_01x03_Male, Connector_PinHeader_2.54mm:PinHeader_1x03_P2.54mm_Vertical, symbol Connector:Conn_01x03_Male
- J20, J21, J22: value Conn_02x09_Odd_Even -> Conn_02x10_Odd_Even; footprint Connector_PinSocket_2.54mm:PinSocket_2x09_P2.54mm_Vertical -> Connector_PinSocket_2.54mm:PinSocket_2x10_P2.54mm_Vertical; symbol Connector_Generic:Conn_02x09_Odd_Even -> Connector_Generic:Conn_02x10_Odd_Even
Connections:
- net A0: now also J20.6 (Pin_6), J21.6 (Pin_6), J22.6 (Pin_6); no longer J20.4 (Pin_4), J21.4 (Pin_4), J22.4 (Pin_4)
- net A1: now also J20.8 (Pin_8), J21.8 (Pin_8), J22.8 (Pin_8); no longer J20.6 (Pin_6), J21.6 (Pin_6), J22.6 (Pin_6)
- net A2: now also J20.10 (Pin_10), J21.10 (Pin_10), J22.10 (Pin_10); no longer J20.8 (Pin_8), J21.8 (Pin_8), J22.8 (Pin_8)
- net CLK: now also J20.1 (Pin_1), J21.1 (Pin_1), J22.1 (Pin_1)
- net D0: now also J20.17 (Pin_17), J21.17 (Pin_17), J22.17 (Pin_17); no longer J20.15 (Pin_15), J21.15 (Pin_15), J22.15 (Pin_15)
- net D1: now also J20.15 (Pin_15), J21.15 (Pin_15), J22.15 (Pin_15); no longer J20.13 (Pin_13), J21.13 (Pin_13), J22.13 (Pin_13)
- net D2: now also J20.13 (Pin_13), J21.13 (Pin_13), J22.13 (Pin_13); no longer J20.11 (Pin_11), J21.11 (Pin_11), J22.11 (Pin_11)
- net D3: now also J20.11 (Pin_11), J21.11 (Pin_11), J22.11 (Pin_11); no longer J20.9 (Pin_9), J21.9 (Pin_9), J22.9 (Pin_9)
- net D4: now also J20.9 (Pin_9), J21.9 (Pin_9), J22.9 (Pin_9); no longer J20.7 (Pin_7), J21.7 (Pin_7), J22.7 (Pin_7)
- net D5: now also J20.7 (Pin_7), J21.7 (Pin_7), J22.7 (Pin_7); no longer J20.5 (Pin_5), J21.5 (Pin_5), J22.5 (Pin_5)
- net D6: now also J20.5 (Pin_5), J21.5 (Pin_5), J22.5 (Pin_5); no longer J20.3 (Pin_3), J21.3 (Pin_3), J22.3 (Pin_3)
- net D7: now also J20.3 (Pin_3), J21.3 (Pin_3), J22.3 (Pin_3); no longer J20.1 (Pin_1), J21.1 (Pin_1), J22.1 (Pin_1)
- net DC: now also J13.5 (Pin_5)
- net DIR: now also J23.10 (Pin_10)
- net DRVSA: now also J23.4 (Pin_4)
- net DSKCHG: now also J23.26 (Pin_26)
- net GND: now also J20.20 (Pin_20), J21.20 (Pin_20), J22.20 (Pin_20), J23.1 (Pin_1), J23.11 (Pin_11), J23.13 (Pin_13), J23.15 (Pin_15), J23.17 (Pin_17), J23.19 (Pin_19), J23.21 (Pin_21), J23.23 (Pin_23), J23.25 (Pin_25), J23.3 (Pin_3), J23.5 (Pin_5), J23.7 (Pin_7), J23.9 (Pin_9), J27.1 (Pin_1), J27.3 (Pin_3); no longer J20.18 (Pin_18), J21.18 (Pin_18), J22.18 (Pin_18)
- net INDEX: now also J23.2 (Pin_2)
- net INT: now also J20.14 (Pin_14), J21.14 (Pin_14), J22.14 (Pin_14); no longer J20.12 (Pin_12), J21.12 (Pin_12), J22.12 (Pin_12)
- net M1: now also J20.4 (Pin_4), J21.4 (Pin_4), J22.4 (Pin_4)
- net MOTEA: now also J23.8 (Pin_8)
- net RD0: now also J21.16 (Pin_16); no longer J21.14 (Pin_14)
- net RD1: now also J22.16 (Pin_16); no longer J22.14 (Pin_14)
- net RD2: now also J20.16 (Pin_16); no longer J20.14 (Pin_14)
- net RDATA: now also J23.22 (Pin_22)
- net RESET: now also J20.18 (Pin_18), J21.18 (Pin_18), J22.18 (Pin_18); no longer J20.16 (Pin_16), J21.16 (Pin_16), J22.16 (Pin_16)
- net SIDE1: now also J23.24 (Pin_24)
- net SLOTCS0: now also J21.12 (Pin_12); no longer J21.10 (Pin_10)
- net SLOTCS1: now also J22.12 (Pin_12); no longer J22.10 (Pin_10)
- net SLOTCS2: now also J20.12 (Pin_12); no longer J20.10 (Pin_10)
- net STEP: now also J23.12 (Pin_12)
- net TRK00: now also J23.18 (Pin_18)
- net VCC: now also J27.2 (Pin_2)
- net WDATA: now also J23.14 (Pin_14)
- net WGATE: now also J23.16 (Pin_16)
- net WPT: now also J23.20 (Pin_20)
- net WR0: now also J21.19 (Pin_19); no longer J21.17 (Pin_17)
- net WR1: now also J22.19 (Pin_19); no longer J22.17 (Pin_17)
- net WR2: now also J20.19 (Pin_19); no longer J20.17 (Pin_17)
- net DC3: now reaches J1.3 (Pin_3)
- net DC3: now also J12.5 (Pin_5), J2.3 (Pin_3), J3.3 (Pin_3), J4.3 (Pin_3), J5.3 (Pin_3)
- new net: J25.1 (Pin_1), J26.1 (Pin_1)
- new net: J25.10 (Pin_10), J26.10 (Pin_10)
- new net: J25.11 (Pin_11), J26.11 (Pin_11)
- new net: J25.12 (Pin_12), J26.12 (Pin_12)
- new net: J25.13 (Pin_13), J26.13 (Pin_13)
- new net: J25.14 (Pin_14), J26.14 (Pin_14)
- new net: J25.15 (Pin_15), J26.15 (Pin_15)
- new net: J25.16 (Pin_16), J26.16 (Pin_16)
- new net: J25.2 (Pin_2), J26.2 (Pin_2)
- new net: J25.3 (Pin_3), J26.3 (Pin_3)
- new net: J25.4 (Pin_4), J26.4 (Pin_4)
- new net: J25.5 (Pin_5), J26.5 (Pin_5)
- new net: J25.6 (Pin_6), J26.6 (Pin_6)
- new net: J25.7 (Pin_7), J26.7 (Pin_7)
- new net: J25.8 (Pin_8), J26.8 (Pin_8)
- new net: J25.9 (Pin_9), J26.9 (Pin_9)
- no-connect marks 69 -> 63
Changed lines of the file:
@@
 Text GLabel 4850 6300 2    50   Output ~ 0
 RX_1
-NoConn ~ 1400 6300
 NoConn ~ 1900 5400
-NoConn ~ 2850 5400
 NoConn ~ 3350 5400
-NoConn ~ 4300 5400
 NoConn ~ 4800 5400
-NoConn ~ 5750 5400
 NoConn ~ 6250 5400
 NoConn ~ 4350 6500
@@
 NoConn ~ 3100 7500
 NoConn ~ 2600 7500
-NoConn ~ 8500 9850
 NoConn ~ 8500 9950
-NoConn ~ 9150 9850
 NoConn ~ 9150 9950
 NoConn ~ 6600 6850
@@
 Wire Wire Line
 	6650 22600 7100 22600
-NoConn ~ 1400 5400
 NoConn ~ 15000 4750
 $Comp
-L Connector_Generic:Conn_02x09_Odd_Even J21
+L Connector_Generic:Conn_02x10_Odd_Even J21
 U 1 1 624AFF30
-P 11300 11450
-F 0 "J21" H 11350 12067 50  0000 C CNN
-F 1 "Conn_02x09_Odd_Even" H 11350 11976 50  0000 C CNN
-F 2 "Connector_PinSocket_2.54mm:PinSocket_2x09_P2.54mm_Vertical" H 11300 11450 50  0001 C CNN
-F 3 "~" H 11300 11450 50  0001 C CNN
-	1    11300 11450
+P 11300 11350
+F 0 "J21" H 11350 11967 50  0000 C CNN
+F 1 "Conn_02x10_Odd_Even" H 11350 11876 50  0000 C CNN
+F 2 "Connector_PinSocket_2.54mm:PinSocket_2x10_P2.54mm_Vertical" H 11300 11350 50  0001 C CNN
+F 3 "~" H 11300 11350 50  0001 C CNN
+	1    11300 11350
 	1    0    0    -1
 $EndComp
@@
 	1    0    0    -1
 $EndComp
-Text GLabel 11600 11050 2    50   Input ~ 0
+Text GLabel 11600 10950 2    50   Input ~ 0
 VCC
 Text GLabel 11600 11450 2    50   Input ~ 0
@@
 SLOTCS0
 $Comp
-L Connector_Generic:Conn_02x09_Odd_Even J22
+L Connector_Generic:Conn_02x10_Odd_Even J22
 U 1 1 625583CE
-P 12700 11450
-F 0 "J22" H 12750 12067 50  0000 C CNN
-F 1 "Conn_02x09_Odd_Even" H 12750 11976 50  0000 C CNN
-F 2 "Connector_PinSocket_2.54mm:PinSocket_2x09_P2.54mm_Vertical" H 12700 11450 50  0001 C CNN
-F 3 "~" H 12700 11450 50  0001 C CNN
-	1    12700 11450
+P 12700 11350
+F 0 "J22" H 12750 11967 50  0000 C CNN
+F 1 "Conn_02x10_Odd_Even" H 12750 11876 50  0000 C CNN
+F 2 "Connector_PinSocket_2.54mm:PinSocket_2x10_P2.54mm_Vertical" H 12700 11350 50  0001 C CNN
+F 3 "~" H 12700 11350 50  0001 C CNN
+	1    12700 11350
 	1    0    0    -1
 $EndComp
@@
 	1    0    0    -1
 $EndComp
-Text GLabel 13000 11050 2    50   Input ~ 0
+Text GLabel 13000 10950 2    50   Input ~ 0
 VCC
 Text GLabel 13000 11450 2    50   Input ~ 0
@@
 FIXME RD AND WR GO TO 18 PIN ?  ADD CLK
 $Comp
-L Connector_Generic:Conn_02x09_Odd_Even J20
+L Connector_Generic:Conn_02x10_Odd_Even J20
 U 1 1 62605154
-P 14050 11450
-F 0 "J20" H 14100 12067 50  0000 C CNN
-F 1 "Conn_02x09_Odd_Even" H 14100 11976 50  0000 C CNN
-F 2 "Connector_PinSocket_2.54mm:PinSocket_2x09_P2.54mm_Vertical" H 14050 11450 50  0001 C CNN
-F 3 "~" H 14050 11450 50  0001 C CNN
-	1    14050 11450
+P 14050 11350
+F 0 "J20" H 14100 11967 50  0000 C CNN
+F 1 "Conn_02x10_Odd_Even" H 14100 11876 50  0000 C CNN
+F 2 "Connector_PinSocket_2.54mm:PinSocket_2x10_P2.54mm_Vertical" H 14050 11350 50  0001 C CNN
+F 3 "~" H 14050 11350 50  0001 C CNN
+	1    14050 11350
 	1    0    0    -1
 $EndComp
@@
 	1    0    0    -1
 $EndComp
-Text GLabel 14350 11050 2    50   Input ~ 0
+Text GLabel 14350 10950 2    50   Input ~ 0
 VCC
 Text GLabel 14350 11450 2    50   Input ~ 0
@@
 	7950 19600 7950 19800
 Connection ~ 7950 19800
+Text GLabel 14350 11050 2    50   Input ~ 0
+M1
+Text GLabel 13850 10950 0    50   Input ~ 0
+CLK
+Text GLabel 12500 10950 0    50   Input ~ 0
+CLK
+Text GLabel 13000 11050 2    50   Input ~ 0
+M1
+Text GLabel 11600 11050 2    50   Input ~ 0
+M1
+Text GLabel 11100 10950 0    50   Input ~ 0
+CLK
+Text GLabel 8500 9850 0    50   Output ~ 0
+DC3
+Text GLabel 9150 9850 2    50   Input ~ 0
+DC
+Text GLabel 1400 6300 0    50   Input ~ 0
+DC3
+Text GLabel 1400 5400 0    50   Input ~ 0
+DC3
+Text GLabel 4300 5400 0    50   Input ~ 0
+DC3
+Text GLabel 5750 5400 0    50   Input ~ 0
+DC3
+Text GLabel 2850 5400 0    50   Input ~ 0
+DC3
+$Comp
+L Connector_Generic:Conn_02x13_Odd_Even J23
+U 1 1 62A4C97D
+P 8050 14900
+F 0 "J23" H 8100 15717 50  0000 C CNN
+F 1 "Conn_02x13_Odd_Even" H 8100 15626 50  0000 C CNN
+F 2 "Connector_IDC:IDC-Header_2x13_P2.54mm_Vertical" H 8050 14900 50  0001 C CNN
+F 3 "~" H 8050 14900 50  0001 C CNN
+	1    8050 14900
+	-1   0    0    -1
+$EndComp
+Wire Wire Line
+	8250 14300 8250 14400
+Connection ~ 8250 14400
+Wire Wire Line
+	8250 14400 8250 14500
+Connection ~ 8250 14500
+Wire Wire Line
+	8250 14500 8250 14600
+Connection ~ 8250 14600
+Wire Wire Line
+	8250 14600 8250 14700
+Connection ~ 8250 14700
+Wire Wire Line
+	8250 14700 8250 14800
+Connection ~ 8250 14800
+Wire Wire Line
+	8250 14800 8250 14900
+Connection ~ 8250 14900
+Wire Wire Line
+	8250 14900 8250 15000
+Connection ~ 8250 15000
+Wire Wire Line
+	8250 15000 8250 15100
+Connection ~ 8250 15100
+Wire Wire Line
+	8250 15100 8250 15200
+Connection ~ 8250 15200
+Wire Wire Line
+	8250 15200 8250 15300
+Connection ~ 8250 15300
+Wire Wire Line
+	8250 15300 8250 15400
+Connection ~ 8250 15400
+Wire Wire Line
+	8250 15400 8250 15500
+$Comp
+L power:GND #PWR0150
+U 1 1 62A87907
+P 8250 15500
+F 0 "#PWR0150" H 8250 15250 50  0001 C CNN
+F 1 "GND" H 8255 15327 50  0000 C CNN
+F 2 "" H 8250 15500 50  0001 C CNN
+F 3 "" H 8250 15500 50  0001 C CNN
+	1    8250 15500
+	1    0    0    -1
+$EndComp
+Connection ~ 8250 15500
+NoConn ~ 7750 14500
+Text GLabel 7750 15400 0    50   Input ~ 0
+SIDE1
+Wire Wire Line
+	6650 13550 6650 15300
+Wire Wire Line
+	6650 15300 7750 15300
+Wire Wire Line
+	7750 15200 6900 15200
+Wire Wire Line
+	6900 15200 6900 13450
+Wire Wire Line
+	7750 15100 7150 15100
+Wire Wire Line
+	7150 15100 7150 13350
+Text GLabel 7750 15000 0    50   Input ~ 0
+WGATE
+Text GLabel 7750 14900 0    50   Input ~ 0
+WDATA
+Text GLabel 7750 14800 0    50   Input ~ 0
+STEP
+Text GLabel 7750 14700 0    50   Input ~ 0
+DIR
+Text GLabel 7750 14600 0    50   Input ~ 0
+MOTEA
+Wire Wire Line
+	6400 13750 6400 15500
+Wire Wire Line
+	6400 15500 7750 15500
+Text GLabel 7750 14400 0    50   Input ~ 0
+DRVSA
+Wire Wire Line
+	7400 12450 7400 14300
+Wire Wire Line
+	7400 14300 7750 14300
+$Comp
+L Connector_Generic:Conn_01x16 J25
+U 1 1 62BAD6C7
+P 11050 16700
+F 0 "J25" H 11130 16692 50  0000 L CNN
+F 1 "Conn_01x16" H 11130 16601 50  0000 L CNN
+F 2 "Connector_PinHeader_2.54mm:PinHeader_1x16_P2.54mm_Horizontal" H 11050 16700 50  0001 C CNN
+F 3 "~" H 11050 16700 50  0001 C CNN
+	1    11050 16700
+	1    0    0    -1
+$EndComp
+$Comp
+L Connector_Generic:Conn_01x16 J26
+U 1 1 62BB1325
+P 10650 16700
+F 0 "J26" H 10568 17617 50  0000 C CNN
+F 1 "Conn_01x16" H 10568 17526 50  0000 C CNN
+F 2 "Connector_PinHeader_2.54mm:PinHeader_1x16_P2.54mm_Vertical" H 10650 16700 50  0001 C CNN
+F 3 "~" H 10650 16700 50  0001 C CNN
+	1    10650 16700
+	-1   0    0    -1
+$EndComp
+$Comp
+L Connector:Conn_01x03_Male J27
+U 1 1 62BB463B
+P 9800 16750
+F 0 "J27" H 9772 16774 50  0000 R CNN
+F 1 "Conn_01x03_Male" H 9772 16683 50  0000 R CNN
+F 2 "Connector_PinHeader_2.54mm:PinHeader_1x03_P2.54mm_Vertical" H 9800 16750 50  0001 C CNN
+F 3 "~" H 9800 16750 50  0001 C CNN
+	1    9800 16750
+	-1   0    0    -1
+$EndComp
+$Comp
+L power:GND #PWR0151
+U 1 1 62BCAD78
+P 9600 16850
+F 0 "#PWR0151" H 9600 16600 50  0001 C CNN
+F 1 "GND" H 9605 16677 50  0000 C CNN
+F 2 "" H 9600 16850 50  0001 C CNN
+F 3 "" H 9600 16850 50  0001 C CNN
+	1    9600 16850
+	1    0    0    -1
+$EndComp
+Text GLabel 9600 16750 0    50   Input ~ 0
+VCC
+Wire Wire Line
+	9600 16650 9200 16650
+Wire Wire Line
+	9200 16650 9200 16850
+Wire Wire Line
+	9200 16850 9600 16850
+Connection ~ 9600 16850
 $EndSCHEMATC
